File: pcb/C3-tiny.kicad_pcb (KiCad board)
At the start: 4 copper layers, 20.3 x 34.3 mm, 29 parts, among them J1 USB_C_Receptacle_USB2.0, J2 Conn_01x10_Pin, J3 Conn_01x10_Pin, U1 ESP32-C3-MINI-1, U2 NCP692MN33T2G, U3 SHT31-DIS

Commit message: Removed cap on BOOT. Cleanup some minor errors
Parts:
- removed C1: 0.1uF, Capacitor_SMD:C_0603_1608Metric_Pad1.08x0.95mm_HandSolder
- moved R9 0.45 mm to (36.6, 52.5)
Routing:
- net /BOOT: track 16.3 -> 27.9 mm, vias 0 -> 1
- net GND: track 61.5 -> 60.2 mm, vias 3 -> 4
- net /IO6: track 33.9 -> 33.4 mm
